Commit message: Design v3: rear pusher for unloading onto a conveyor; keep v2 in backup_v2
- CAD: push blade on a T8 lead screw and two 8 mm rods outside the deck
  edges (robot_cad.py); collision check over the whole stroke; 8-sheet
  drawing set; regenerated STEP, STL, DXF, renders, BOM and ROS mesh
- Electrical: third BTS7960, pusher motor and two limit switches on all
  three schematic sheets; GPIO 9/10 (driver) and 4/6 (switches)
- ROS: pusher_node, conveyor docking and unloading in the mission
  (--conveyor), tools/test_pusher.py
- Docs: build guide steps marked "Pusher"; PUSHER_IMPACT.md compares v3
  with v2
- backup_v2/: untouched copy of design v2 (commit 11388c4)

The pusher has not been built or run on hardware yet.

File: robot_ws/src/cargo_bot/urdf/cargo_bot.urdf.xacro (robot description, xacro)
@@ -1,8 +1,9 @@
 <?xml version="1.0"?>
-<!-- Cargo robot model (design v2). All numbers come from cad/robot_cad.py (converted to metres).
+<!-- Cargo robot model (design v3). All numbers come from cad/robot_cad.py (converted to metres).
      Frames: base_footprint (on the floor, under the axle centre) -> base_link (axle centre)
              X = forward, Y = left, Z = up.
      Used by the real robot (robot.launch.py) and by the Gazebo simulation (sim.launch.py, sim:=true).
-     Masses are estimates (total ~5 kg); correct them after weighing the real robot. -->
+     Masses are estimates (total ~6 kg with the pusher); correct them after weighing the real robot.
+     The pusher is part of the body mesh (blade parked); it has no joint and does not move in the model. -->
 <robot name="cargo_bot" xmlns:xacro="http://www.ros.org/wiki/xacro">
   <xacro:arg name="sim" default="false"/>
@@ -12,5 +13,5 @@
   <xacro:property name="wheel_y" value="0.165"/>
   <xacro:property name="wheel_mass" value="0.15"/>
-  <xacro:property name="body_mass" value="4.5"/>
+  <xacro:property name="body_mass" value="5.6"/>
   <!-- RPLIDAR orientation: if obstacles in front show up BEHIND the robot in RViz, change pi to 0.0 -->
   <xacro:property name="laser_yaw" value="${pi}"/>
